File: KXR_pi_hat_v0.2/KXR_pi_hat_v0.2.kicad_pcb (KiCad board)
At the start: 2 copper layers, 65 x 56 mm, 10 parts, among them J1 Conn_01x05_Pin, J2 Conn_01x05_Pin, J3 Conn_01x05_Pin, J4 Conn_01x05_Pin, U2 Raspberry_Pi_2_3

Commit message: Finishing touches and production files
Parts:
- added CS: SolderJumper_3_Open, Jumper:SolderJumper-3_P1.3mm_Open_RoundedPad1.0x1.5mm_NumberLabels, B.Cu at (71.0, 105.2)
- added DRDY: SolderJumper_3_Open, Jumper:SolderJumper-3_P1.3mm_Open_RoundedPad1.0x1.5mm_NumberLabels, B.Cu at (71.0, 87.8)
- added G***: LOGO, Library:KXR_logo, B.Cu at (96.7, 93.3)
- added PDWN: SolderJumper_3_Open, Jumper:SolderJumper-3_P1.3mm_Open_RoundedPad1.0x1.5mm_NumberLabels, B.Cu at (71.0, 96.5)
- U1: renamed from U2; moved to B.Cu
- moved U1 48.3 mm to (116.6, 74.8)
Connections:
- ADS1256 Breakout pad 6: /DRDY_1 -> Net-(JP1-C)
- ADS1256 Breakout pad 7: /CS_1 -> Net-(JP2-C)
- ADS1256 Breakout pad 8: /PDWN_1 -> Net-(JP3-C)
- U1 pad 15: unconnected-(U2-GPIO22-Pad15) -> /DRDY_1
- U1 pad 16: unconnected-(U2-GPIO23-Pad16) -> /DRDY_2
- U1 pad 18: /DRDY_1 -> /PDWN_1
- U1 pad 22: /PDWN_1 -> /PDWN_2
- U1 pad 29: unconnected-(U2-GCLK1/GPIO5-Pad29) -> /R1
- U1 pad 31: unconnected-(U2-GCLK2/GPIO6-Pad31) -> /R2
- U1 pad 32: unconnected-(U2-PWM0/GPIO12-Pad32) -> /LED
- U1 pad 33: unconnected-(U2-PWM1/GPIO13-Pad33) -> /R3
- U1 pad 35: unconnected-(U2-GPIO19/MISO1-Pad35) -> /R5
- U1 pad 36: unconnected-(U2-GPIO16-Pad36) -> /R4
- U1 pad 37: unconnected-(U2-GPIO26-Pad37) -> /R8
- U1 pad 38: unconnected-(U2-GPIO20/MOSI1-Pad38) -> /R6
- U1 pad 40: unconnected-(U2-GPIO21/SCLK1-Pad40) -> /R7
Routing:
- net /CS_2: track 0.00 -> 46.6 mm, vias 0 -> 2
- net /PDWN_2: track 0.00 -> 35.8 mm, vias 0 -> 1
- net /DRDY_2: track 0.00 -> 23.9 mm, vias 0 -> 2
- net Net-(JP1-C): track 0.00 -> 18.4 mm, vias 0 -> 1
- net Net-(JP3-C): track 0.00 -> 15.6 mm
- net /DRDY_1: track 39.1 -> 24.1 mm
- net /PDWN_1: track 47.2 -> 32.5 mm
- net Net-(JP2-C): track 0.00 -> 10.5 mm
- net +5V: track 104.9 -> 111.6 mm
- net /CS_1: track 47.0 -> 45.2 mm, vias 0 -> 2
- net /LC1_S+: track 59.1 -> 58.4 mm
- net /LC2_S+: track 43.8 -> 43.1 mm
- net /LC2_S-: track 47.4 -> 46.7 mm
- net /LC3_S+: track 28.6 -> 27.9 mm
- net /LC3_S-: track 32.1 -> 31.5 mm
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Other:
- board text added: "4-Channel Differential ADS1256 Data Acquisition Board for Pi"
- board text added: "Launch Test Infrastructure"
