File: KXR_pi_hat_v0.2/KXR_pi_hat_v0.2.kicad_sch (KiCad schematic)
At the start: 6 parts, among them J1 Conn_01x05_Pin, J2 Conn_01x05_Pin, J3 Conn_01x05_Pin, J4 Conn_01x05_Pin, U2 Raspberry_Pi_2_3

Commit message: Finishing touches and production files
Parts:
- added JP1, JP2, JP3: SolderJumper_3_Open, Jumper:SolderJumper-3_P1.3mm_Open_RoundedPad1.0x1.5mm_NumberLabels, symbol Jumper:SolderJumper_3_Open
- renumbered U2 to U1, U1 to U2
Connections:
- net CS_1: now also JP2.1 (A); no longer U2.7 (CS)
- net CS_2: now also JP2.3 (B)
- net DRDY_1: now also U1.15 (GPIO22), JP1.1 (A); no longer U1.18 (GPIO24), U2.6 (DRDY)
- net PDWN_1: now also U1.18 (GPIO24), JP3.1 (A); no longer U1.22 (GPIO25), U2.8 (PDWN)
- net DRDY_2: now reaches U1.16 (GPIO23)
- net DRDY_2: now also JP1.3 (B)
- net R1: now reaches U1.29 (GCLK1/GPIO5)
- net R2: now reaches U1.31 (GCLK2/GPIO6)
- net LED: now reaches U1.32 (PWM0/GPIO12)
- net R3: now reaches U1.33 (PWM1/GPIO13)
- net R5: now reaches U1.35 (GPIO19/MISO1)
- net R4: now reaches U1.36 (GPIO16)
- net R8: now reaches U1.37 (GPIO26)
- net R6: now reaches U1.38 (GPIO20/MOSI1)
- net R7: now reaches U1.40 (GPIO21/SCLK1)
- new net: JP2.2 (C), U2.7 (CS)
- new net: JP3.2 (C), U2.8 (PDWN)
- new net: JP1.2 (C), U2.6 (DRDY)
- new net PDWN_2: JP3.3 (B), U1.22 (GPIO25)
- no-connect marks 23 -> 12
Other:
- moved on the sheet: J1, J2, J3, J4, U1, U2

Commit message: Added README, clarified schematic
Parts:
- U1: value Raspberry_Pi_2_3 -> Raspberry Pi
- U2: value ~ -> HiLetgo ADS1256 Module
Connections:
- net LED: no longer names the net of U1.32 (PWM0/GPIO12)
- net R1: no longer names the net of U1.29 (GCLK1/GPIO5)
- net R2: no longer names the net of U1.31 (GCLK2/GPIO6)
- net R3: no longer names the net of U1.33 (PWM1/GPIO13)
- net R4: no longer names the net of U1.36 (GPIO16)
- net R5: no longer names the net of U1.35 (GPIO19/MISO1)
- net R6: no longer names the net of U1.38 (GPIO20/MOSI1)
- net R7: no longer names the net of U1.40 (GPIO21/SCLK1)
- net R8: no longer names the net of U1.37 (GPIO26)
- no-connect marks 12 -> 21
Other:
- note added: "4x JST S4B-XH-A"
Changed lines of the file:
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@@
 		(rev "v0.2")
+	)
+	(text "4x JST S4B-XH-A"
+		(exclude_from_sim no)
+		(at 177.8 62.992 0)
+		(effects
+			(font
+				(size 1.27 1.27)
+			)
+		)
 	)
 	(junction
@@
 	)
 	(no_connect
+		(at 73.66 115.57)
+	)
+	(no_connect
 		(at 73.66 90.17)
 	)
@@
 	)
 	(no_connect
+		(at 73.66 95.25)
+	)
+	(no_connect
 		(at 73.66 118.11)
+	)
+	(no_connect
+		(at 73.66 85.09)
 	)
 	(no_connect
@@
 	)
 	(no_connect
+		(at 73.66 100.33)
+	)
+	(no_connect
+		(at 114.3 97.79)
+	)
+	(no_connect
 		(at 114.3 77.47)
 	)
@@
 	)
 	(no_connect
+		(at 73.66 97.79)
+	)
+	(no_connect
+		(at 114.3 120.65)
+	)
+	(no_connect
+		(at 114.3 95.25)
+	)
+	(no_connect
 		(at 73.66 77.47)
 	)
+	(no_connect
+		(at 114.3 118.11)
+	)
 	(wire
 		(pts
@@
 	(wire
 		(pts
-			(xy 116.84 95.25) (xy 114.3 95.25)
-		)
-		(stroke
-			(width 0)
-			(type default)
-		)
-	)
-	(wire
-		(pts
-			(xy 71.12 100.33) (xy 73.66 100.33)
-		)
-		(stroke
-			(width 0)
-			(type default)
-		)
-	)
-	(wire
-		(pts
 			(xy 114.3 102.87) (xy 116.84 102.87)
 		)
@@
 	(wire
 		(pts
-			(xy 71.12 95.25) (xy 73.66 95.25)
-		)
-		(stroke
-			(width 0)
-			(type default)
-		)
-	)
-	(wire
-		(pts
 			(xy 212.09 100.33) (xy 214.63 100.33)
 		)
@@
 	(wire
 		(pts
-			(xy 116.84 120.65) (xy 114.3 120.65)
-		)
-		(stroke
-			(width 0)
-			(type default)
-		)
-	)
-	(wire
-		(pts
 			(xy 157.48 102.87) (xy 171.45 102.87)
 		)
@@
 	(wire
 		(pts
-			(xy 71.12 85.09) (xy 73.66 85.09)
-		)
-		(stroke
-			(width 0)
-			(type default)
-		)
-	)
-	(wire
-		(pts
 			(xy 143.51 77.47) (xy 144.78 77.47)
 		)
@@
 	(wire
 		(pts
-			(xy 116.84 97.79) (xy 114.3 97.79)
-		)
-		(stroke
-			(width 0)
-			(type default)
-		)
-	)
-	(wire
-		(pts
 			(xy 189.23 72.39) (xy 190.5 72.39)
 		)
@@
 	(wire
 		(pts
-			(xy 71.12 97.79) (xy 73.66 97.79)
-		)
-		(stroke
-			(width 0)
-			(type default)
-		)
-	)
-	(wire
-		(pts
 			(xy 71.12 110.49) (xy 73.66 110.49)
 		)
@@
 	(wire
 		(pts
-			(xy 71.12 115.57) (xy 73.66 115.57)
-		)
-		(stroke
-			(width 0)
-			(type default)
-		)
-	)
-	(wire
-		(pts
 			(xy 212.09 80.01) (xy 213.36 80.01)
 		)
@@
 		(pts
 			(xy 142.24 132.08) (xy 149.86 132.08)
-		)
-		(stroke
-			(width 0)
-			(type default)
-		)
-	)
-	(wire
-		(pts
-			(xy 116.84 118.11) (xy 114.3 118.11)
 		)
 		(stroke
@@
 		)
 	)
-	(label "R8"
-		(at 71.12 115.57 180)
-		(effects
-			(font
-				(size 1.27 1.27)
-			)
-			(justify right bottom)
-		)
-	)
 	(label "LC4_S-"
 		(at 212.09 77.47 180)
@@
 		)
 	)
-	(label "R1"
-		(at 116.84 95.25 0)
-		(effects
-			(font
-				(size 1.27 1.27)
-			)
-			(justify left bottom)
-		)
-	)
 	(label "LC3_S+"
 		(at 189.23 74.93 180)
@@
 		)
 	)
-	(label "R4"
-		(at 71.12 85.09 180)
-		(effects
-			(font
-				(size 1.27 1.27)
-			)
-			(justify right bottom)
-		)
-	)
 	(label "LC4_S+"
 		(at 212.09 74.93 180)
@@
 		)
 	)
-	(label "R2"
-		(at 116.84 97.79 0)
-		(effects
-			(font
-				(size 1.27 1.27)
-			)
-			(justify left bottom)
-		)
-	)
 	(label "LC4_S+"
 		(at 214.63 118.11 0)
@@
 		)
 	)
-	(label "R3"
-		(at 116.84 120.65 0)
-		(effects
-			(font
-				(size 1.27 1.27)
-			)
-			(justify left bottom)
-		)
-	)
 	(label "DRDY_1"
 		(at 71.12 105.41 180)
@@
 		)
 	)
-	(label "R5"
-		(at 71.12 95.25 180)
-		(effects
-			(font
-				(size 1.27 1.27)
-			)
-			(justify right bottom)
-		)
-	)
 	(label "LC1_S+"
 		(at 143.51 74.93 180)
@@
 		)
 	)
-	(label "R7"
-		(at 71.12 100.33 180)
-		(effects
-			(font
-				(size 1.27 1.27)
-			)
-			(justify right bottom)
-		)
-	)
 	(label "LC2_S-"
 		(at 166.37 77.47 180)
@@
 		)
 	)
-	(label "R6"
-		(at 71.12 97.79 180)
-		(effects
-			(font
-				(size 1.27 1.27)
-			)
-			(justify right bottom)
-		)
-	)
 	(label "LC3_S+"
 		(at 214.63 113.03 0)
@@
 	(label "CS_1"
 		(at 138.43 120.65 0)
-		(effects
-			(font
-				(size 1.27 1.27)
-			)
-			(justify left bottom)
-		)
-	)
-	(label "LED"
-		(at 116.84 118.11 0)
 		(effects
 			(font
@@
 			)
 		)
-		(property "Value" "~"
+		(property "Value" "HiLetgo ADS1256 Module"
 			(at 191.77 96.52 0)
 			(effects
@@
 			)
 		)
-		(property "Value" "Raspberry_Pi_2_3"
+		(property "Value" "Raspberry Pi"
 			(at 96.1741 135.89 0)
 			(effects
